File: components/sockets/pcb/sockets.brd (EAGLE design)
At the start: 69.2 x 54.7 mm, 10 parts, among them IC1 7805T

Commit message: Worked on pcbs
Parts:
- C1: device rcl:C025-050X050 -> capacitor-wima:C5B2.5
- moved X1 2.30 mm to (35.5, 14.3)
- moved C1 1.50 mm to (41.0, 24.4)
Routing:
- net N$6: track 43.7 -> 46.6 mm
- net GND: track 75.1 -> 77.4 mm
- net N$9: track 0.00 -> 1.20 mm
Changed lines of the file:
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@@
 </autorouter>
 <elements>
-<element name="X1" library="con-conrad" package="733980-62" value="" x="35.52" y="16.58" rot="R270"/>
+<element name="X1" library="con-conrad" package="733980-62" value="" x="35.52" y="14.28" rot="R270"/>
 <element name="TRANSMITTER" library="pinhead" package="1X04" value="" x="36.72" y="41.04" rot="R270"/>
 <element name="JP1" library="pinhead" package="1X08" value="" x="64.56" y="58.12"/>
@@
 <element name="JP6" library="pinhead" package="1X06" value="" x="88.9" y="9.19"/>
 <element name="IC1" library="linear" package="TO220H" value="7805T" x="57.4" y="28.7" rot="MR90"/>
-<element name="C1" library="rcl" package="C025-050X050" value="330n" x="41.1" y="25.9" rot="R90"/>
+<element name="C1" library="capacitor-wima" package="C5B2.5" value="330n" x="41" y="24.4" rot="R90"/>
 <element name="C2" library="rcl" package="C025-050X050" value="100n" x="41.1" y="31.8" rot="R90"/>
 <element name="ANTENNA" library="con-coax" package="BU-SMA-G" value="BU-SMA-G" x="36.7" y="53" rot="R180">
@@
 <contactref element="C1" pad="2"/>
 <contactref element="C2" pad="1"/>
-<wire x1="41.09" y1="11.58" x2="37.78" y2="16.18" width="1.5" layer="1"/>
+<wire x1="41.09" y1="9.28" x2="37.78" y2="16.18" width="1.5" layer="1"/>
 <contactref element="TRANSMITTER" pad="2"/>
 <contactref element="JP1" pad="2"/>
@@
 <wire x1="40.9" y1="27.8" x2="41.1" y2="27.8" width="1.5" layer="16"/>
 <wire x1="41.1" y1="27.8" x2="41.1" y2="28.8" width="1.5" layer="16"/>
-<wire x1="41.1" y1="27.17" x2="41.3" y2="27.17" width="1.5" layer="16"/>
+<wire x1="41" y1="26.94" x2="41.3" y2="27.17" width="1.5" layer="16"/>
 <wire x1="41.3" y1="27.17" x2="41.3" y2="28.6" width="1.5" layer="16"/>
-<wire x1="41.1" y1="27.17" x2="41.2" y2="27.17" width="1.5" layer="16"/>
+<wire x1="41" y1="26.94" x2="41.2" y2="27.17" width="1.5" layer="16"/>
 <wire x1="41.2" y1="27.17" x2="41.2" y2="28.7" width="1.5" layer="16"/>
 <wire x1="47.24" y1="28.7" x2="51.5" y2="28.7" width="1.5" layer="16"/>
@@
 <wire x1="40.9" y1="44.2" x2="39.9" y2="44.2" width="1.5" layer="16"/>
 <wire x1="39.9" y1="44.2" x2="39.9" y2="51.4" width="1.5" layer="16"/>
+<wire x1="41.1" y1="28.8" x2="41.1" y2="30.53" width="0" layer="19" extent="16-16"/>
 </signal>
 <signal name="N$4">
@@
 <contactref element="IC1" pad="1"/>
 <contactref element="C1" pad="1"/>
-<wire x1="44.09" y1="16.58" x2="42.3" y2="11.18" width="1.5" layer="1"/>
-<wire x1="44.09" y1="16.58" x2="47.24" y2="16.58" width="1.5" layer="16"/>
+<wire x1="44.09" y1="14.28" x2="42.3" y2="11.18" width="1.5" layer="1"/>
 <contactref element="TRANSMITTER" pad="4"/>
-<wire x1="41.1" y1="24.63" x2="47.24" y2="24.63" width="1.5" layer="16"/>
 <wire x1="47.24" y1="24.63" x2="47.24" y2="26.16" width="1.5" layer="16"/>
 <wire x1="36.72" y1="37.23" x2="37" y2="37.23" width="1.5" layer="16"/>
 <wire x1="37" y1="37.23" x2="37" y2="36.8" width="1.5" layer="16"/>
 <wire x1="37" y1="36.8" x2="36.7" y2="36.8" width="1.5" layer="16"/>
-<wire x1="36.7" y1="36.8" x2="36.7" y2="24.63" width="1.5" layer="16"/>
-<wire x1="41.1" y1="24.63" x2="36.7" y2="24.63" width="1.5" layer="16"/>
-<wire x1="47.24" y1="16.58" x2="47.24" y2="26.16" width="1.5" layer="16"/>
+<wire x1="36.7" y1="36.8" x2="36.7" y2="21.86" width="1.5" layer="16"/>
+<wire x1="47.24" y1="14.28" x2="47.24" y2="21.86" width="1.5" layer="16"/>
+<wire x1="47.24" y1="22.1" x2="47.24" y2="26.16" width="1.5" layer="16"/>
+<wire x1="44.09" y1="14.28" x2="47.24" y2="14.28" width="1.5" layer="16"/>
+<wire x1="41" y1="21.86" x2="36.7" y2="21.86" width="1.5" layer="16"/>
+<wire x1="41" y1="21.86" x2="47.24" y2="21.86" width="1.5" layer="16"/>
+<wire x1="47.24" y1="21.86" x2="47.24" y2="22.1" width="1.5" layer="16"/>
 </signal>
 <signal name="N$41">
@@
 <wire x1="36.7" y1="44.85" x2="36.7" y2="53" width="1" layer="16"/>
 </signal>
+<signal name="N$9">
+<wire x1="41.1" y1="30.7" x2="42.2" y2="30.7" width="1.5" layer="16"/>
+<wire x1="42.2" y1="30.7" x2="42.2" y2="30.6" width="1.5" layer="16"/>
+</signal>
 </signals>
