File: components/ambilight/pcb/ambilight.sch (EAGLE design)
At the start: 12 parts, among them IC1 7805TV

Commit message: Interface work
Parts:
- TB, TG, TR: value foo -> IRF740
Changed lines of the file:
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@@
 </classes>
 <parts>
-<part name="TR" library="transistor-power" deviceset="IRF740" device="" value="foo"/>
-<part name="TG" library="transistor-power" deviceset="IRF740" device="" value="foo"/>
-<part name="TB" library="transistor-power" deviceset="IRF740" device="" value="foo"/>
+<part name="TR" library="transistor-power" deviceset="IRF740" device="" value="IRF740"/>
+<part name="TG" library="transistor-power" deviceset="IRF740" device="" value="IRF740"/>
+<part name="TB" library="transistor-power" deviceset="IRF740" device="" value="IRF740"/>
 <part name="X1" library="con-conrad" deviceset="73398?" device="0-62"/>
 <part name="AURORA" library="pinhead" deviceset="PINHD-1X4" device=""/>
